Commit message: qarm_v2: coarse-arm/fine-gripper primitive collisions with buried-primitive pruning (43 -> 32), via shared collision_simplify
Co-Authored-By: Claude Opus 5.5 <noreply@anthropic.com>

File: models/qarm_v2/qarm_with_gripper.urdf (robot description, URDF)
Before this commit: robot QARM, 12 links, 11 joints
Links:
- link BICEP: geometry collision box size=0.07148836 0.07938018 0.1010919; collision cylinder length=0.02758156 radius=0.03723188
- link END-EFFECTOR: geometry collision cylinder length=0.0148 radius=0.0177; visual mesh filename=meshes/visual/END-EFFECTOR.stl
- link FOREARM: geometry collision box size=0.02469205 0.04413417 0.09927912; collision box size=0.06530222 0.06939311 0.07617549
- link Link1A: geometry collision box size=0.005409164 0.01985234 0.05049457; collision box size=0.01909041 0.02061038 0.0363732
- link Link1B: geometry collision box size=0.0051625 0.005741029 0.01643748; collision box size=0.01476701 0.01726665 0.01854675
- link Link2A: geometry collision box size=0.0217 0.02303058 0.05918772; visual mesh filename=meshes/visual/LINK2A.stl
- link Link2B: geometry collision box size=0.0217 0.02303058 0.05918772; visual mesh filename=meshes/visual/LINK2B.stl
- link YAW: geometry collision box size=0.04868893 0.0677309 0.152806; collision cylinder length=0.02026642 radius=0.07145107
- link base_link: geometry collision box size=0.09586612 0.295675 0.335675; visual mesh filename=meshes/visual/base_link.stl
- link gripper_base_link: geometry collision box size=0.009530679 0.01521615 0.0342406; collision box size=0.01180058 0.03423404 0.03900235
